File: hardware/CPU_board/CPU_board.kicad_pcb (KiCad board)
At the start: 4 copper layers, 51.2 x 25.8 mm, 111 parts, among them J1 TF TF-018 1.5mm, J2 SOUTH, J3 NORTH, J4 Conn_01x6_Male, J5 Conn_01x03, J6 JTAG, J8 Conn_01x10_Male, U1 EA3036A, U2 W25Q32JVZPIQ, U3 D1s-eLQFP128, U4 PAD30, U5 PAD30, U6 PAD30, U7 PAD30, U8 PAD30, U9 PAD30, X1 24MHz, X2 32.768KHz

Commit message: fixed mixup of pins G5/G4 (3rd diff pair ODD) and DE/PCLK (3rd diff pair EVEN), now with correct polarity for diff pairs
Parts:
- added R32: 10k, Resistor_SMD:R_0402_1005Metric, B.Cu at (101.6, 103.3)
- added R35: 10k, Resistor_SMD:R_0402_1005Metric, B.Cu at (101.6, 102.3)
- added R36: 10k, Resistor_SMD:R_0402_1005Metric, B.Cu at (105.2, 111.0)
- added R40: 10k, Resistor_SMD:R_0402_1005Metric, B.Cu at (106.2, 111.0)
- moved R30 3.79 mm to (107.0, 105.5)
- moved C37 3.05 mm to (105.0, 113.7), turned to -90 degrees
- moved C2 1.88 mm to (106.2, 113.9), turned to 90 degrees
- moved G*** 1.56 mm to (103.8, 102.9)
- moved R21 0.41 mm to (99.7, 105.2)
- moved C4 0.40 mm to (99.7, 106.1)
- moved C7 0.38 mm to (99.7, 104.2)
- moved C5 0.38 mm to (99.7, 103.3)
- moved C35 0.31 mm to (101.9, 109.9)
- moved C32 0.25 mm to (100.0, 109.9)
Connections:
- J2 pad 3: /LCD_V3P -> /LCD_V3N
- J2 pad 5: /LCD_V3N -> /LCD_V3P
- J3 pad 3: /LCD_U3P -> /LCD_U3N
- J3 pad 5: /LCD_U3N -> /LCD_U3P
Routing:
- net GND: track 210.5 -> 189.6 mm, vias 55 -> 54
- net 3V3: track 213.4 -> 226.3 mm
- net /PSEL: track 23.2 -> 13.5 mm
- net /SDA2: track 8.75 -> 12.4 mm
- net VSYS: track 24.0 -> 21.8 mm
- net /SCK: track 24.1 -> 22.4 mm
- net /SDA: track 24.8 -> 23.2 mm
- net /SCK2: track 8.59 -> 10.2 mm
- net /LCD_V3N: track 15.9 -> 14.4 mm
- net /LCD_D9: track 18.7 -> 17.8 mm
- net /X32KIN: track 6.42 -> 5.52 mm
- net /TP-Y2: track 24.7 -> 25.5 mm
- net /LCD_D8: track 19.7 -> 20.5 mm
- net /LCD_U3P: track 13.3 -> 14.1 mm
- net /LCD_V3P: track 14.0 -> 14.6 mm
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Other:
- board text added: "CPU board v0.11"
- board text added: "CUPRUMFLOW"
- board text removed: "CPU board"
- board text removed: "Memory Card"
