File: hardware/CPU_board/CPU_board.kicad_sch (KiCad schematic)
At the start: 101 parts, among them J1 TF 1.5H 短体, J2 DF12NB_3.0_-30DS-0.5V_51, J3 DF12NB_3.0_-30DS-0.5V_51, J4 JTAG, J5 Conn_01x03, J6 Conn_01x6_Male, U1 EA3036A, U2 W25Q32JVZPIQ, U3 D1s-eLQFP128, U5 PAD30, U6 PAD30, U7 PAD30, X1 24MHz, X2 32.768KHz

Commit message: update PCB design files
Connections:
- net PSEL: now reaches J2.9, R26.1
Changed lines of the file:
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@@
+		)
+	)
+	(label "PSEL"
+		(at 146.05 231.14 180)
+		(fields_autoplaced yes)
+		(effects
+			(font
+				(size 1.27 1.27)
+			)
+			(justify right bottom)
 		)
 	)

Commit message: update PCB design files
Parts:
- removed C2: 0.1uF, Capacitor_SMD:C_0402_1005Metric, symbol GRM188B30J106ME47D_12
- removed C36: 0.1uF, Library:C_0402_1005Metric, symbol Periph-altium-import:0_CAP
- removed C41: 0.1uF, Capacitor_SMD:C_0402_1005Metric, symbol GRM188B30J106ME47D
- removed C42: 10u, Capacitor_SMD:C_0603_1608Metric, symbol C_0402_US
- removed C44: 0.1uF, Capacitor_SMD:C_0402_1005Metric, symbol GRM188B30J106ME47D_8
- removed J4: JTAG, Connector:Tag-Connect_TC2030-IDC-NL_2x03_P1.27mm_Vertical, symbol PRT-12807:PRT-12807
- removed J6: Conn_01x6_Male, Connector_PinHeader_2.54mm:PinHeader_1x06_P2.54mm_Vertical, symbol Connector_Generic:Conn_01x06
- removed R1, R11, R13, R17: 47k, Resistor_SMD:R_0402_1005Metric, symbol R_0201_EU_2
- removed R18: 84.5K 1%, Library:R_0402_1005Metric, symbol Device:R
- removed R26: 10K, Library:R_0402_1005Metric, symbol D1s-altium-import:2_RES
- removed R27: 5K1, Resistor_SMD:R_0402_1005Metric, symbol R_0603_EU_5
- removed R29: 5K1, Resistor_SMD:R_0402_1005Metric, symbol R_0603_EU_4
- added C2: 10u, Capacitor_SMD:C_0603_1608Metric, symbol C_0402_US_1
- added C36: 0.1uF, Capacitor_SMD:C_0402_1005Metric, symbol GRM188B30J106ME47D_8
- added C41: 0.1uF, Capacitor_SMD:C_0402_1005Metric, symbol GRM188B30J106ME47D
- added D2: D_Schottky, Library:U-DFN1608-2_L1.6-W0.8-RD, symbol Device:D_Schottky
- added J4: Conn_01x6_Male, Connector_PinHeader_2.54mm:PinHeader_1x06_P2.54mm_Vertical, symbol Connector_Generic:Conn_01x06
- added J6: JTAG, Connector:Tag-Connect_TC2030-IDC-NL_2x03_P1.27mm_Vertical, symbol PRT-12807:PRT-12807
- added J8: Conn_01x10_Male, Connector_PinHeader_2.54mm:PinHeader_1x10_P2.54mm_Vertical, symbol Connector_Generic:Conn_01x10
- added JP1: SolderJumper_3_Bridged12, Jumper:SolderJumper-3_P1.3mm_Bridged12_RoundedPad1.0x1.5mm, symbol Jumper:SolderJumper_3_Bridged12
- added R1, R11, R13, R17: 47k, Resistor_SMD:R_0402_1005Metric, symbol R_0201_EU_1
- added R18: 100k, Resistor_SMD:R_0402_1005Metric, symbol R_0603_EU_1
- added R26: 84.5K 1%, Library:R_0402_1005Metric, symbol Device:R
- added R27: 5K1, Resistor_SMD:R_0402_1005Metric, symbol R_0603_EU_4
- added R29: 5K1, Resistor_SMD:R_0402_1005Metric, symbol R_0603_EU_5
- added R30: 10K, Library:R_0402_1005Metric, symbol D1s-altium-import:2_RES
- added R31: 10k, Resistor_SMD:R_0402_1005Metric, symbol R_0402_EU_20
- added R33, R34: 22, Resistor_SMD:R_0402_1005Metric, symbol R_0603_EU_9
- added U4: PAD30, TestPoint:TestPoint_Pad_D1.0mm, symbol PAD30
- added U8: PAD30, TestPoint:TestPoint_Pad_D1.0mm, symbol PAD30_1
- added U9: PAD30, TestPoint:TestPoint_Pad_D1.0mm, symbol PAD30_2
- FEL1: value EVQPUJ_EVQPUA -> FEL; footprint Button_Switch_SMD:Panasonic_EVQPUJ_EVQPUA -> Button_Switch_SMD:SW_SPST_PTS810; MPN (none) -> PTS810SJM250SMTRLFS
- J1: value TF 1.5H 短体 -> TF TF-018 1.5mm; footprint TFCARD 短体 1.5H -> Library:TF-SMD_TF-018; MPN (none) -> TF-018
- J2: value DF12NB_3.0_-30DS-0.5V_51 -> SOUTH; LCSC Part Number C5148308 -> (none); MFG (none) -> Hirose; MPN (none) -> DF12NB(3.0)-30DS-0.5V(51); Manufacturer_Name Hirose -> (none); Manufacturer_Part_Number DF12NB(3.0)-30DS-0.5V(51) -> (none)
- J3: value DF12NB_3.0_-30DS-0.5V_51 -> NORTH; LCSC Part Number C5148308 -> (none); MFG (none) -> Hirose; MPN (none) -> DF12NB(3.0)-30DS-0.5V(51); Manufacturer_Name Hirose -> (none); Manufacturer_Part_Number DF12NB(3.0)-30DS-0.5V(51) -> (none)
- LED1: value LED-0603_R -> LED-0603_BLUE; footprint (none) -> LED_SMD:LED_0603_1608Metric; LCSC Part Number (none) -> C7429915; MPN (none) -> NCD0603B5
- LED2: value LED-0603_R -> LED-0603_PURPLE; footprint (none) -> LED_SMD:LED_0603_1608Metric; LCSC Part Number (none) -> C7371898; MPN (none) -> XL-1608UVC-04
- R22: value 5k1 -> 3k3
- R25, R28: LCSC Part Number C171671 -> (none); MPN (none) -> FRC0402F1053TS
- RESET1: value EVQPUJ_EVQPUA -> RESET; footprint Button_Switch_SMD:Panasonic_EVQPUJ_EVQPUA -> Button_Switch_SMD:SW_SPST_PTS810; MPN (none) -> PTS810SJM250SMTRLFS
- U1: footprint Package_DFN_QFN:WQFN-20-1EP_3x3mm_P0.4mm_EP1.7x1.7mm -> Package_DFN_QFN:QFN-20-1EP_3x3mm_P0.4mm_EP1.65x1.65mm; MPN (none) -> EA3036CQBR
- U3: LCSC Part Nuber ALT (none) -> C5197687; LCSC Part Number (none) -> C5365285; MFG (none) -> Allwinner Tech; MPN (none) -> D1s; MPN_ALT (none) -> T113-S3
- USB1, USB2: footprint USB-C-SMD_TYPEC-304-BCP16 -> Connector_USB:USB_C_Receptacle_G-Switch_GT-USB-7010ASV; LCSC Part Number C720629 -> (none); MFG XUNPU -> G-Switch; MPN TYPEC-304-BCP16 -> GT-USB-7010ASV
Connections:
- net PE0 is gone; now on net SCK2: U3.44 (PE0)
- net PE1 is gone; now on net SDA2: U3.45 (PE1)
- net PE8 is gone; now on net PSEL: U3.39 (PE8)
- net 0V9: now also U9.1
- net 1V8A: now also C36.1
- net 1V8_DRAM: now also U8.1
- net 3V3: now also C2.2, D2.2 (A), J4.6 (Pin_6), J6.1, J8.10 (Pin_10), JP1.3 (B), R1.1, R11.1, R13.1, R17.1, R30.2, U4.1
- net CTS1: now also J4.1 (Pin_1)
- net GND: now also C2.1, C36.2, C41.1, J4.5 (Pin_5), J6.5, J8.8 (Pin_8), R26.1, R27.2, R29.1, R31.1; no longer J2.28, J2.30
- net JTAG_TCK: now also J6.4
- net JTAG_TDI: now also J6.3
- net JTAG_TDO: now also J6.6
- net JTAG_TMS: now also J6.2
- net LCD_D16: now also J2.28; no longer J3.28
- net LCD_D17: now also J2.30; no longer J3.30
- net PSEL: now also R30.1
- net RST: now also J8.7 (Pin_7)
- net RTS1: now also J4.4 (Pin_4)
- net RX1: now also J4.3 (Pin_3)
- net SCK: no longer J5.2 (Pin_2)
- net SCK2: no longer U3.35 (PE2)
- net SDA: no longer J5.1 (Pin_1)
- net SDA2: no longer U3.33 (PE3)
- net SDC0_D0: now also R11.2
- net SDC0_D1: now also R1.2
- net SDC0_D2: now also R17.2
- net SDC0_D3: now also R13.2
- net TX1: now also J4.2 (Pin_2)
- net VBUS: now also J8.9 (Pin_9), JP1.1 (A), R18.1; no longer C11.2, C12.2, U1.16 (VCC), U1.19 (VIN3), U1.7 (VIN2), U1.8 (EN2), U1.9 (EN1)
- net at J2.21: now also R26.2
- net at R24.1: now also USB2.B5 (CC2); no longer USB1.B5 (CC2)
- net at USB2.A5 (CC1): now also R23.2
- net at USB1.A5 (CC1): now also R29.2; no longer R23.2
- net LDO_BOUT: now reaches U3.30 (LDOB-OUT)
- net LDO_BOUT: now also C41.2
- net PG1: now reaches U3.118 (PG1)
- net PG1: now also J8.2 (Pin_2)
- net PG2: now reaches U3.119 (PG2)
- net PG2: now also J8.3 (Pin_3)
- net PG0: now reaches U3.120 (PG0)
- net PG0: now also J8.1 (Pin_1)
- net PG3: now reaches U3.121 (PG3)
- net PG3: now also J8.4 (Pin_4)
- net PG5: now reaches U3.122 (PG5)
- net PG5: now also J8.6 (Pin_6)
- net PG4: now reaches U3.123 (PG4)
- net PG4: now also J8.5 (Pin_5)
- net D0+ renamed USB_D0+
- net D0- renamed USB_D0-
- net D1+ renamed USB_D1+
- net D1- renamed USB_D1-
- net LCD_CLK renamed LCD_U3N
- net LCD_U3N: now also U3.76 (PD19); no longer U3.75 (PD18)
- net LCD_D10 renamed LCD_CKP
- net LCD_D11 renamed LCD_CKN
- net LCD_D12 renamed LCD_V3P
- net LCD_D13 renamed LCD_V3N
- net LCD_D14 renamed LCD_U0P
- net LCD_D15 renamed LCD_U0N
- net LCD_D18 renamed LCD_U1P
- net LCD_D19 renamed LCD_U1N
- net LCD_D2 renamed LCD_V0P
- net LCD_D20 renamed LCD_U2P
- net LCD_D21 renamed LCD_U2N
- net LCD_D22 renamed LCD_UCKP
- net LCD_D23 renamed LCD_UCKN
- net LCD_D3 renamed LCD_V0N
- net LCD_D4 renamed LCD_V1P
- net LCD_D5 renamed LCD_V1N
- net LCD_D6 renamed LCD_V2P
- net LCD_V2P: now also R34.2
- net LCD_D7 renamed LCD_V2N
- net LCD_V2N: now also R33.2
- net LCD_DE renamed LCD_U3P
- net LCD_U3P: now also U3.75 (PD18); no longer U3.76 (PD19)
- net SPI0_D0 renamed SDC2_D0
- net SDC2_D0: now also R37.2, U2.3 (/WP-IO2); no longer U2.5 (DI)
- net SPI0_D1 renamed SDC2_D1
- net SPI0_D2 renamed SDC2_D2
- net SDC2_D2: now also U2.5 (DI-IO0), R31.2; no longer R37.2, U2.3 (/WP)
- net SPI0_D3 renamed SDC2_D3
- new net: R18.2, U1.9 (EN1)
- new net: R27.1, USB1.B5 (CC2)
- new net B6: J3.28, R34.1
- new net B7: J3.30, R33.1
- new net RX0: J5.1 (Pin_1), U3.33 (PE3)
- new net TX0: J5.2 (Pin_2), U3.35 (PE2)
- new net VSYS: C11.2, C12.2, D2.1 (K), JP1.2 (C), U1.16 (VCC), U1.19 (VIN3), U1.7 (VIN2), U1.8 (EN2)
- no-connect marks 29 -> 23
Other:
- note added: "CPU board, based on: YuzukiNezha D1s RISC-V Linux Core (Company: YuzukiHD) Originally drawn by GloomyGhost https://oshwhub.com/GloomyGhost/yuzukif133 https://github.com/YuzukiHD/YuzukiNezha-D1s LICENSE: CERN Open Hardware License"
- note added: "DISP"
- note added: "Headers & JTAG"
- note added: "LCD_CLK LCD_DE"
- note added: "LCD_DE LCD_CLK"
- note added: "LVDS0-V3P LCD0-D12 LVDS0-V3N LCD0-D13"
- note added: "LVDS1-CKP(D22-R6) LVDS1-CKN(D23-R7) LVDS1-V2P(D20-R4) LVDS1-V2N(D21-R5) LVDS1-V1P(D18-R2) LVDS1-V1N(D19-R3) LVDS1-V0P(D14-G6) LVDS1-V0N(D15-G7)"
- note added: "LVDS1-V3P LCD0-CLK LVDS1-V3N LCD0-DE"
- note added: "LVDSO-CKP(D10-G2) LVDSO-CKN(D11-G3) LVDSO-V2P(D6-B6) LVDSO-V2N(D7-B7) LVDSO-V1P(D4-B4) LVDSO-V1N(D5-B5) LVDSO-V0P(D2-B2) LVDSO-V0N(D3-B3)"
- note added: "MOSI= BOOTSEL0"
- note added: "NORTH"
- note added: "NORTH Connector"
- note added: "PADS"
- note added: "PC5: SEL1/SPI0_D1/MISO PC4: SEL0/SPI0_D2/MOSI SEL[1:0]: 00: NOR > NAND 01: SD > NOR > Other √10: SD > NAND > Other 11 SD0 > EMMC2 > EMMC2_USR >Other"
- note added: "PSEL"
- note added: "Pin 20"
- note added: "SEL[1:0] 00: NOR > NAND 01: SD > NOR > Other √10: SD > NAND > Other 11 SD > EMMC2 > EMMC2_USR >Other"
- note added: "SOUTH"
- note added: "SOUTH Connector"
- note added: "SPI0 CS/MOSI/MISO has reset PU"
- note added: "USB 1 OTG"
- note added: "USB 2 HOST"
- note added: "Video connectors"
- note added: "XTAL"
- note removed: "3.5MM PAD"
- note removed: "CPU board, based on: YuzukiNezha D1s RISC-V Linux Core (Company: YuzukiHD) Originally drawn by GloomyGhost https://oshwhub.com/GloomyGhost/yuzukif133 https://github.com/YuzukiHD/YuzukiNezha-D1 LICENSE: CERN-OHL"
- note removed: "Connectors"
- note removed: "EA3036 may not be enough, try it first"
- note removed: "North connector"
- note removed: "South connector"
- note removed: "USB 1"
- note removed: "USB 2"
- company: (none) -> (C) 2023-2024 Victor Suarez Rovere
- title: (none) -> CPU board
- moved on the sheet: C1, C16, C17, C18, C19, C20, C21, C22, C30, C38, C40, C43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
