File: hardware/FPGA_board/decopling.kicad_sch (KiCad schematic)
At the start: 24 parts

Commit message: update PCB design files
Parts:
- C48, C49, C52, C53, C56, C58, C60, C62, C63, C66, C67, C74: MPN (none) -> GRM033R61C103KA12D; PN GRM033R61C103KA12D -> (none)
- C50, C51, C54, C55, C57, C59, C61, C64, C65, C68, C69, C75: MPN (none) -> CL03A104KQ3NNNC; PN CL03A104KQ3NNNC -> (none)
Other:
- company: (none) -> (C) 2023-2026 Victor Suarez Rovere
- title: (none) -> FPGA board
Changed lines of the file:
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@@
 	(generator_version "8.0")
 	(paper "A4")
+	(title_block
+		(title "FPGA board")
+		(date "2026-03-16")
+		(rev "0.1")
+		(company "(C) 2023-2026 Victor Suarez Rovere")
+		(comment 1 "Based on OrangeCrab board r0.1")
+		(comment 2 "https://github.com/orangecrab-fpga/orangecrab-hardware/tree/main/hardware/orangecrab_r0.1")
+		(comment 3 "﻿CERN Open Hardware Licence v1.2 ")
+	)
 	(junction
 		(at 59.69 62.23)
@@
 			)
 		)
-		(property "PN" "GRM033R61C103KA12D"
+		(property "MPN" "GRM033R61C103KA12D"
 			(at 33.02 34.29 0)
 			(effects
@@
 			)
 		)
-		(property "PN" "CL03A104KQ3NNNC"
+		(property "MPN" "CL03A104KQ3NNNC"
 			(at 38.1 34.29 0)
 			(effects
@@
 			)
 		)
-		(property "PN" "GRM033R61C103KA12D"
+		(property "MPN" "GRM033R61C103KA12D"
 			(at 54.61 34.29 0)
 			(effects
@@
 			)
 		)
-		(property "PN" "CL03A104KQ3NNNC"
+		(property "MPN" "CL03A104KQ3NNNC"
 			(at 59.69 34.29 0)
 			(effects
@@
 			)
 		)
-		(property "PN" "GRM033R61C103KA12D"
+		(property "MPN" "GRM033R61C103KA12D"
 			(at 76.2 34.29 0)
 			(effects
@@
 			)
 		)
-		(property "PN" "CL03A104KQ3NNNC"
+		(property "MPN" "CL03A104KQ3NNNC"
 			(at 81.28 34.29 0)
 			(effects
@@
 			)
 		)
-		(property "PN" "GRM033R61C103KA12D"
+		(property "MPN" "GRM033R61C103KA12D"
 			(at 97.79 34.29 0)
 			(effects
@@
 			)
 		)
-		(property "PN" "CL03A104KQ3NNNC"
+		(property "MPN" "CL03A104KQ3NNNC"
 			(at 102.87 34.29 0)
 			(effects
@@
 			)
 		)
-		(property "PN" "GRM033R61C103KA12D"
+		(property "MPN" "GRM033R61C103KA12D"
 			(at 118.11 34.29 0)
 			(effects
@@
 			)
 		)
-		(property "PN" "CL03A104KQ3NNNC"
+		(property "MPN" "CL03A104KQ3NNNC"
 			(at 123.19 34.29 0)
 			(effects
@@
 			)
 		)
-		(property "PN" "GRM033R61C103KA12D"
+		(property "MPN" "GRM033R61C103KA12D"
 			(at 33.02 67.31 0)
 			(effects
@@
 			)
 		)
-		(property "PN" "CL03A104KQ3NNNC"
+		(property "MPN" "CL03A104KQ3NNNC"
 			(at 38.1 67.31 0)
 			(effects
@@
 			)
 		)
-		(property "PN" "GRM033R61C103KA12D"
+		(property "MPN" "GRM033R61C103KA12D"
 			(at 54.61 67.31 0)
 			(effects
@@
 			)
 		)
-		(property "PN" "CL03A104KQ3NNNC"
+		(property "MPN" "CL03A104KQ3NNNC"
 			(at 59.69 67.31 0)
 			(effects
@@
 			)
 		)
-		(property "PN" "GRM033R61C103KA12D"
+		(property "MPN" "GRM033R61C103KA12D"
 			(at 97.79 67.31 0)
 			(effects
@@
 			)
 		)
-		(property "PN" "CL03A104KQ3NNNC"
+		(property "MPN" "CL03A104KQ3NNNC"
 			(at 102.87 67.31 0)
 			(effects
@@
 			)
 		)
-		(property "PN" "GRM033R61C103KA12D"
+		(property "MPN" "GRM033R61C103KA12D"
 			(at 119.38 67.31 0)
 			(effects
@@
 			)
 		)
-		(property "PN" "CL03A104KQ3NNNC"
+		(property "MPN" "CL03A104KQ3NNNC"
 			(at 124.46 67.31 0)
 			(effects
@@
 			)
 		)
-		(property "PN" "GRM033R61C103KA12D"
+		(property "MPN" "GRM033R61C103KA12D"
 			(at 97.79 96.52 0)
 			(effects
@@
 			)
 		)
-		(property "PN" "CL03A104KQ3NNNC"
+		(property "MPN" "CL03A104KQ3NNNC"
 			(at 102.87 96.52 0)
 			(effects
@@
 			)
 		)
-		(property "PN" "GRM033R61C103KA12D"
+		(property "MPN" "GRM033R61C103KA12D"
 			(at 119.38 96.52 0)
 			(effects
@@
 			)
 		)
-		(property "PN" "CL03A104KQ3NNNC"
+		(property "MPN" "CL03A104KQ3NNNC"
 			(at 124.46 96.52 0)
 			(effects
@@
 			)
 		)
-		(property "PN" "GRM033R61C103KA12D"
+		(property "MPN" "GRM033R61C103KA12D"
 			(at 142.24 96.52 0)
 			(effects
@@
 			)
 		)
-		(property "PN" "CL03A104KQ3NNNC"
+		(property "MPN" "CL03A104KQ3NNNC"
 			(at 147.32 96.52 0)
 			(effects
