File: hardware/FPGA_board/fileFPGA.kicad_sch (KiCad schematic)
At the start: 11 parts, among them J6 JTAG, U3 ECP5U25, U6 XT25Q08DDTIGT

Commit message: update PCB design files
Parts:
- removed U6: XT25Q08DDTIGT, gkl_housings_dfn:DFN-8-1EP_3x2mm_Pitch0.5mm, symbol OrangeCrab-rescue:AT25SF081-gkl_mem
- added U6: W25Q128JVPIQ, Package_SON:WSON-8-1EP_6x5mm_P1.27mm_EP3.4x4.3mm, symbol Memory_Flash:W25Q128JVS
- C1, C19, C25: MPN (none) -> GRM033R61C103KA12D; PN GRM033R61C103KA12D -> (none)
- C20, C26, C4: MPN (none) -> CL03A104KQ3NNNC; PN CL03A104KQ3NNNC -> (none)
- OSC1: MPN (none) -> OT252048MJBA4SL; PN OT252048MJBA4SL -> (none)
- R27: MPN (none) -> RC0201FR-074K7L; PN RC0201FR-074K7L -> (none)
- U3: value ECP5U25 -> ECP5; MFG (none) -> Lattice Semiconductor Corporation; MPN (none) -> LFE5U-85F-8MG285I; Mfg Lattice Semiconductor Corporation -> (none); PN LFE5U-25F-8MG285C -> (none); SN-DK LFE5UM-25F-6MG285C-ND -> (none)
Connections:
- net GND: now also U6.4 (GND), U6.9 (THERMAL)
- net P3.3V: now also U6.8 (VCC)
- net QSPI_D2: now also U6.3 (IO2)
- net QSPI_D3: now also U6.7 (IO3)
- net SPI_CONFIG_MISO: now also U6.2 (DO(IO1))
- net SPI_CONFIG_MOSI: now also U6.5 (DI(IO0))
- net SPI_CONFIG_SCK: now also U6.6 (CLK)
- net SPI_CONFIG_SS: now also U6.1 (~{CS})
- net USB_PULLUP renamed PULLUP_USB
Other:
- note added: "1V35"
- note removed: "1V5"
- company: (none) -> (C) 2023-2026 Victor Suarez Rovere
- title: (none) -> FPGA board
- moved on the sheet: C19, C20, U3F, U3G, U3I
