File: hardware/FPGA_board/fileHyperRAM.kicad_sch (KiCad schematic)
At the start: 32 parts, among them U4 MT41K64M16TW-107_J-TR

Commit message: update PCB design files
Parts:
- C21, C22, C34, C35, C36, C37: MPN (none) -> JMK105C6105KV-F; PN JMK105C6105KV-F -> (none)
- C23, C24: MPN (none) -> GRM188R60J226MEA0D; PN GRM188R60J226MEA0D -> (none)
- C27, C38, C40, C42, C44, C45: MPN (none) -> GRM033R61C103KA12D; PN GRM033R61C103KA12D -> (none)
- C30, C31, C32, C33, C39, C41, C43: MPN (none) -> CL03A104KQ3NNNC; PN CL03A104KQ3NNNC -> (none)
- FB2, FB3: MPN (none) -> BLM15AG601SN1D; PN BLM15AG601SN1D -> (none)
- R19: MPN (none) -> RC0402FR-07240RL; PN RC0402FR-07240RL -> (none)
- R3: MPN (none) -> RC0201FR-070RL; PN RC0201FR-070RL -> (none)
- RN1, RN2, RN3, RN4, RN5, RN6: MPN (none) -> WA04X49R9FTL; PN WA04X49R9FTL -> (none)
- U4: MPN (none) -> MT41K64M16TW-107:J TR; PN MT41K64M16TW-107:J TR -> (none)
Connections:
- net GND: now also U4.G8 (VSS)
- no-connect marks 3 -> 7
Other:
- company: (none) -> (C) 2023-2026 Victor Suarez Rovere
- title: (none) -> FPGA board
Changed lines of the file:
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@@
 	(paper "A4")
 	(title_block
-		(date "2024-04-20")
+		(title "FPGA board")
+		(date "2026-03-16")
+		(rev "0.1")
+		(company "(C) 2023-2026 Victor Suarez Rovere")
+		(comment 1 "Based on OrangeCrab board r0.1")
+		(comment 2 "https://github.com/orangecrab-fpga/orangecrab-hardware/tree/main/hardware/orangecrab_r0.1")
+		(comment 3 "﻿CERN Open Hardware Licence v1.2 ")
 	)
 	(junction
@@
 	)
 	(no_connect
+		(at 199.39 161.29)
+	)
+	(no_connect
 		(at 179.07 111.76)
 	)
 	(no_connect
+		(at 194.31 161.29)
+	)
+	(no_connect
+		(at 191.77 161.29)
+	)
+	(no_connect
 		(at 179.07 106.68)
 	)
@@
 		(at 179.07 109.22)
 	)
+	(no_connect
+		(at 196.85 161.29)
+	)
 	(wire
 		(pts
@@
 	(wire
 		(pts
+			(xy 229.87 140.97) (xy 213.36 140.97)
+		)
+		(stroke
+			(width 0)
+			(type default)
+		)
+	)
+	(wire
+		(pts
 			(xy 104.14 55.88) (xy 104.14 58.42)
 		)
@@
 			)
 		)
-		(property "PN" "MT41K64M16TW-107:J TR"
+		(property "MPN" "MT41K64M16TW-107:J TR"
 			(at 195.58 104.14 0)
 			(effects
@@
 		(pin "T9"
 		)
+		(pin "G8"
+		)
+		(pin "L9"
+		)
+		(pin "J1"
+		)
+		(pin "J9"
+		)
+		(pin "L1"
+		)
 		(instances
 			(project "FPGA_board"
@@
 			)
 		)
-		(property "PN" "RC0201FR-070RL"
+		(property "MPN" "RC0201FR-070RL"
 			(at 124.46 124.46 0)
 			(effects
@@
 			)
 		)
-		(property "PN" "JMK105C6105KV-F"
+		(property "MPN" "JMK105C6105KV-F"
 			(at 207.01 55.88 0)
 			(effects
@@
 			)
 		)
-		(property "PN" "JMK105C6105KV-F"
+		(property "MPN" "JMK105C6105KV-F"
 			(at 212.09 55.88 0)
 			(effects
@@
 			)
 		)
-		(property "PN" "CL03A104KQ3NNNC"
+		(property "MPN" "CL03A104KQ3NNNC"
 			(at 184.15 55.88 0)
 			(effects
@@
 			)
 		)
-		(property "PN" "CL03A104KQ3NNNC"
+		(property "MPN" "CL03A104KQ3NNNC"
 			(at 189.23 55.88 0)
 			(effects
@@
 			)
 		)
-		(property "PN" "JMK105C6105KV-F"
+		(property "MPN" "JMK105C6105KV-F"
 			(at 207.01 36.83 0)
 			(effects
@@
 			)
 		)
-		(property "PN" "JMK105C6105KV-F"
+		(property "MPN" "JMK105C6105KV-F"
 			(at 212.09 36.83 0)
 			(effects
@@
 			)
 		)
-		(property "PN" "CL03A104KQ3NNNC"
+		(property "MPN" "CL03A104KQ3NNNC"
 			(at 184.15 36.83 0)
 			(effects
@@
 			)
 		)
-		(property "PN" "CL03A104KQ3NNNC"
+		(property "MPN" "CL03A104KQ3NNNC"
 			(at 189.23 36.83 0)
 			(effects
@@
 			)
 		)
-		(property "PN" "GRM033R61C103KA12D"
+		(property "MPN" "GRM033R61C103KA12D"
 			(at 104.14 38.1 0)
 			(effects
@@
 			)
 		)
-		(property "PN" "CL03A104KQ3NNNC"
+		(property "MPN" "CL03A104KQ3NNNC"
 			(at 104.14 62.23 0)
 			(effects
@@
 			)
 		)
-		(property "PN" "GRM033R61C103KA12D"
+		(property "MPN" "GRM033R61C103KA12D"
 			(at 110.49 38.1 0)
 			(effects
@@
 			)
 		)
-		(property "PN" "CL03A104KQ3NNNC"
+		(property "MPN" "CL03A104KQ3NNNC"
 			(at 110.49 62.23 0)
 			(effects
@@
 			)
 		)
-		(property "PN" "GRM033R61C103KA12D"
+		(property "MPN" "GRM033R61C103KA12D"
 			(at 121.92 38.1 0)
 			(effects
@@
 			)
 		)
-		(property "PN" "CL03A104KQ3NNNC"
+		(property "MPN" "CL03A104KQ3NNNC"
 			(at 121.92 62.23 0)
 			(effects
@@
 			)
 		)
-		(property "PN" "GRM033R61C103KA12D"
+		(property "MPN" "GRM033R61C103KA12D"
 			(at 105.41 97.79 0)
 			(effects
@@
 			)
 		)
-		(property "PN" "GRM033R61C103KA12D"
+		(property "MPN" "GRM033R61C103KA12D"
 			(at 111.76 97.79 0)
 			(effects
@@
 			)
 		)
-		(property "PN" "RC0402FR-07240RL"
+		(property "MPN" "RC0402FR-07240RL"
 			(at 228.6 96.52 0)
 			(effects
@@
 			)
 		)
-		(property "PN" "JMK105C6105KV-F"
+		(property "MPN" "JMK105C6105KV-F"
 			(at 250.19 55.88 0)
 			(effects
@@
 			)
 		)
-		(property "PN" "GRM188R60J226MEA0D"
+		(property "MPN" "GRM188R60J226MEA0D"
 			(at 255.27 55.88 0)
 			(effects
@@
 			)
 		)
-		(property "PN" "BLM15AG601SN1D"
+		(property "MPN" "BLM15AG601SN1D"
 			(at 260.35 49.53 0)
 			(effects
@@
 			)
 		)
-		(property "PN" "JMK105C6105KV-F"
+		(property "MPN" "JMK105C6105KV-F"
 			(at 250.19 82.55 0)
 			(effects
@@
 			)
 		)
-		(property "PN" "GRM188R60J226MEA0D"
+		(property "MPN" "GRM188R60J226MEA0D"
 			(at 255.27 82.55 0)
 			(effects
@@
 			)
 		)
-		(property "PN" "BLM15AG601SN1D"
+		(property "MPN" "BLM15AG601SN1D"
 			(at 260.35 76.2 0)
 			(effects
@@
 			)
 		)
-		(property "PN" "WA04X49R9FTL"
+		(property "MPN" "WA04X49R9FTL"
 			(at 67.31 45.72 0)
 			(effects
@@
 			)
 		)
-		(property "PN" "WA04X49R9FTL"
+		(property "MPN" "WA04X49R9FTL"
 			(at 67.31 60.96 0)
 			(effects
@@
 			)
 		)
-		(property "PN" "WA04X49R9FTL"
+		(property "MPN" "WA04X49R9FTL"
 			(at 67.31 76.2 0)
 			(effects
@@
 			)
 		)
-		(property "PN" "WA04X49R9FTL"
+		(property "MPN" "WA04X49R9FTL"
 			(at 67.31 91.44 0)
 			(effects
@@
 			)
 		)
-		(property "PN" "WA04X49R9FTL"
+		(property "MPN" "WA04X49R9FTL"
 			(at 67.31 106.68 0)
 			(effects
@@
 			)
 		)
-		(property "PN" "WA04X49R9FTL"
+		(property "MPN" "WA04X49R9FTL"
 			(at 67.31 121.92 0)
 			(effects
@@
 			)
 		)
-		(property "PN" "GRM033R61C103KA12D"
+		(property "MPN" "GRM033R61C103KA12D"
 			(at 52.07 123.19 0)
 			(effects
@@
 					(unit 1)
 				)
+			)
+		)
+	)
+	(symbol
+		(lib_id "OrangeCrab-rescue:GND-gkl_power")
+		(at 229.87 140.97 0)
+		(unit 1)
+		(exclude_from_sim no)
+		(in_bom yes)
+		(on_board yes)
+		(dnp no)
+		(property "Reference" "#PWR015"
+			(at 229.87 147.32 0)
+			(effects
+				(font
+					(size 1.27 1.27)
+				)
+				(hide yes)
+			)
+		)
+		(property "Value" "GND"
+			(at 229.9462 144.1704 0)
+			(effects
+				(font
+					(size 1.27 1.27)
+				)
+			)
+		)
+		(property "Footprint" ""
+			(at 227.33 149.86 0)
+			(effects
+				(font
+					(size 1.27 1.27)
+				)
+				(hide yes)
+			)
+		)
+		(property "Datasheet" ""
+			(at 229.87 140.97 0)
+			(effects
+				(font
+					(size 1.27 1.27)
+				)
+				(hide yes)
+			)
+		)
+		(property "Description" ""
+			(at 229.87 140.97 0)
+			(effects
+				(font
+					(size 1.27 1.27)
+				)
+				(hide yes)
+			)
+		)
+		(pin "1"
+		)
+		(instances
+			(project "FPGA_board"
+				(path "/66670491-5507-4d5c-bc12-3561ec3542a1/00000000-0000-0000-0000-00005abd38f2"
+					(reference "#PWR015")
+					(unit 1)
+				)
