File: hardware/FPGA_board/fileIO.kicad_sch (KiCad schematic)
At the start: 38 parts, among them J1 USB_C_Receptacle_USB2.0, J2 Conn_01x6_Male, J3 USB_C_Receptacle_USB2.0, J5 Conn_01x03, J7 Conn_02x15_Odd_Even, J8 Conn_02x15_Odd_Even, SW1 SW_Push

Commit message: update PCB design files
Parts:
- removed J7, J8: Conn_02x15_Odd_Even, gkl_conn:DF12(3.0)-30DP-0.5V(86), symbol Connector_Generic:Conn_02x15_Odd_Even
- removed TP19, TP20, TP3, TP4: SMD_TP, gkl_misc:TestPoint_Pad_D0.5mm, symbol Connector:TestPoint_Flag
- added J10: Conn_01x04, Connector_PinHeader_2.54mm:PinHeader_1x04_P2.54mm_Vertical, symbol Connector_Generic:Conn_01x04
- added J4: Conn_01x04_Male, Connector_PinHeader_2.54mm:PinHeader_1x04_P2.54mm_Vertical, symbol Connector_Generic:Conn_01x04
- added J7, J8: Conn_02x15_Odd_Even, Library:DF12NB3030DP05V51, symbol Connector_Generic_MountingPin:Conn_02x15_Odd_Even_MountingPin
- added R31, R32: 22, Resistor_SMD:R_0402_1005Metric, symbol R_0603_EU_9
- C76: MPN (none) -> CL03A104KQ3NNNC; PN CL03A104KQ3NNNC -> (none)
- D1: MPN (none) -> MHPA1010RGBDT; PN MHPA1010RGBDT -> (none)
- R10, R9: value 51K -> 12K
- R11, R12: Mfg ‎Yageo‎ -> (none)
- R20: MPN (none) -> RC0201FR-071K5L; PN RC0201FR-071K5L -> (none)
- R21, R22, R23, R24, R26, R4: MPN (none) -> RC0201FR-074K7L; PN RC0201FR-074K7L -> (none)
- R29: footprint Resistor_SMD:R_0201_0603Metric -> Resistor_SMD:R_0402_1005Metric; MPN (none) -> 0402WGF2103TCE; Mfg ‎Yageo‎ -> (none)
- SW1: footprint gkl_misc:PTS_810_SMT_Switch -> Button_Switch_SMD:SW_SPST_PTS810; MPN (none) -> PTS810SJM250SMTRLFS; PN PTS810SJM250SMTRLFS -> (none)
- TP1, TP2, TP26, TP27: footprint gkl_misc:TestPoint_Pad_D0.5mm -> TestPoint:TestPoint_Pad_D1.0mm
- TP28, TP29, TP30, TP31, TP32, TP33: footprint gkl_misc:TestPoint_Pad_D0.5mm -> Library:TestPoint_Pad_D0.5mm
- USBD1: renamed from J1; MPN (none) -> GT-USB-7010ASV; PN GT-USB-7010ASV -> (none)
- USBH1: renamed from J3; MPN (none) -> GT-USB-7010ASV; Mfg (none) -> G-Switch
Connections:
- net AUX_0+: now also J8.6 (Pin_6)
- net AUX_0-: now also J8.4 (Pin_4)
- net AUX_1+: now also J8.12 (Pin_12), R31.2
- net AUX_1-: now also J8.10 (Pin_10), R32.2
- net AUX_2+: now also J8.18 (Pin_18)
- net AUX_2-: now also J8.16 (Pin_16)
- net AUX_3+: now also J7.6 (Pin_6)
- net AUX_3-: now also J7.4 (Pin_4)
- net AUX_4+: now also J8.5 (Pin_5)
- net AUX_4-: now also J8.3 (Pin_3)
- net AUX_5+: now also J8.17 (Pin_17)
- net AUX_5-: now also J8.15 (Pin_15)
- net AUX_6+: now also J8.22 (Pin_22)
- net AUX_6-: now also J8.24 (Pin_24)
- net FPGA_RESET: now also J10.4 (Pin_4)
- net GND: now also J10.3 (Pin_3), J7.14 (Pin_14), J7.2 (Pin_2), J7.20 (Pin_20), J7.25 (Pin_25), J7.26 (Pin_26), J7.8 (Pin_8), J7.MP (MountPin), J8.14 (Pin_14), J8.2 (Pin_2), J8.20 (Pin_20), J8.25 (Pin_25), J8.26 (Pin_26), J8.28 (Pin_28), J8.30 (Pin_30), J8.8 (Pin_8), J8.MP (MountPin); no longer R10.2, R9.2
- net HPD/ID: now also J8.21 (Pin_21)
- net IO_0: now also J2.3 (Pin_3); no longer J2.2 (Pin_2)
- net IO_1: now also J2.2 (Pin_2); no longer J2.1 (Pin_1)
- net IO_10: now also J4.1 (Pin_1), J7.18 (Pin_18)
- net IO_11: now also J7.1 (Pin_1), J7.10 (Pin_10)
- net IO_12: now also J7.12 (Pin_12), J7.7 (Pin_7)
- net IO_13: now also J4.4 (Pin_4), J7.5 (Pin_5)
- net IO_5: now also J7.19 (Pin_19), J7.22 (Pin_22)
- net IO_6: now also J7.13 (Pin_13), J7.24 (Pin_24)
- net IO_9: now also J4.2 (Pin_2), J7.16 (Pin_16)
- net IO_MISO: now also J2.1 (Pin_1); no longer J2.3 (Pin_3)
- net IO_SCK: now also J4.3 (Pin_3), J7.3 (Pin_3)
- net IO_SCL: now also J5.1 (Pin_1), J7.17 (Pin_17); no longer J5.2 (Pin_2)
- net IO_SDA: now also J5.2 (Pin_2), J7.15 (Pin_15); no longer J5.1 (Pin_1)
- net LED_B: now also J7.11 (Pin_11)
- net LED_G: now also R22.1; no longer R23.1
- net LED_R: now also R23.1; no longer R22.1
- net P3.3V: now also R10.1, R9.1, J10.1 (Pin_1), J7.27 (Pin_27), J7.29 (Pin_29), J8.27 (Pin_27), J8.29 (Pin_29)
- net PUSB_VBUS: now also J10.2 (Pin_2), J7.23 (Pin_23), J8.23 (Pin_23)
- net SPI_0: now also J8.9 (Pin_9)
- net SPI_1: now also J8.11 (Pin_11)
- net at USBH1.A5 (CC1): now also R9.2; no longer R9.1
- net at R30.1: now also J7.21 (Pin_21)
- net at R26.1: now also J7.9 (Pin_9)
- net at USBH1.B5 (CC2): now also R10.2; no longer R10.1
- net USB_PULLUP renamed PULLUP_USB
- new net: J7.28 (Pin_28), R32.1
- new net: J7.30 (Pin_30), R31.1
- no-connect marks 0 -> 4
Other:
- note added: "+3V3 GND RTS# RX TX CTS#"
- note added: "DISP"
- note added: "HOST-only USB pulldowns"
- note added: "LVDS0-V3P LCD0-D12 LVDS0-V3N LCD0-D13"
- note added: "LVDS1-CKP(D22-R6) LVDS1-CKN(D23-R7) LVDS1-V2P(D20-R4) LVDS1-V2N(D21-R5) LVDS1-V1P(D18-R2) LVDS1-V1N(D19-R3) LVDS1-V0P(D14-G6) LVDS1-V0N(D15-G7)"
- note added: "LVDS1-V3P LCD0-CLK LVDS1-V3N LCD0-DE"
- note added: "LVDSO-CKP(D10-G2) LVDSO-CKN(D11-G3) LVDSO-V2P(D6-B6) LVDSO-V2N(D7-B7) LVDSO-V1P(D4-B4) LVDSO-V1N(D5-B5) LVDSO-V0P(D2-B2) LVDSO-V0N(D3-B3)"
- note added: "NORTH Connector"
- note added: "NOTES: https://hackaday.com/2023/08/07/all-about-usb-c-example-circuits https://cdn.sparkfun.com/assets/e/b/4/f/7/USB-C_Datasheet.pdf"
- note added: "OTG from ULX3S"
- note added: "PSEL"
- note added: "SOUTH Connector"
- note added: "TODO: add DEBUG UART"
- note removed: "+3V3 GND I/O - MOSI I/O - MISO I/O - RX I/O - TX"
- note removed: "HOST-only USB"
- company: (none) -> (C) 2023-2026 Victor Suarez Rovere
- title: (none) -> FPGA board
- moved on the sheet: R21, R26, R29, R30, TP1, TP2
