File: hardware/FPGA_board/filePOWER.kicad_sch (KiCad schematic)
At the start: 35 parts, among them U1 RY1303 or EA3036, U10 NCP115-2.5, U8 TPS51206

Commit message: update PCB design files
Parts:
- removed U10: NCP115-2.5, gkl_housings_son:X2SON_4_1.0x1.0mm, symbol OrangeCrab-rescue:NCP167-gkl_pmic
- added C13: 100pF, Capacitor_SMD:C_0201_0603Metric, symbol Device:C
- added C28: 4.7uF, Capacitor_SMD:C_0402_1005Metric, symbol Device:C
- added D2: D_Schottky, Library:U-DFN1608-2_L1.6-W0.8-RD, symbol Device:D_Schottky
- added JP1, JP2: SolderJumper_3_Bridged12, Jumper:SolderJumper-3_P1.3mm_Bridged12_RoundedPad1.0x1.5mm, symbol Jumper:SolderJumper_3_Bridged12
- added L4: 2.2uH, Library:Murata_DFE201612P-2R2M=P2, symbol Periph-altium-import:0_L
- added R33: 15k, Resistor_SMD:R_0201_0603Metric, symbol Device:R
- added R34: 4.7k, Resistor_SMD:R_0201_0603Metric, symbol Device:R
- added U2: TLV62569APDRL, Package_TO_SOT_SMD:SOT-563, symbol Regulator_Switching:TLV62569DRL
- added U7: NCP115AMX250TCG, Package_DFN_QFN:OnSemi_XDFN4-1EP_1.0x1.0mm_EP0.52x0.52mm, symbol Regulator_Linear:NCP115AMX250TCG
- C10: MPN (none) -> CL03A224MQ3NNNC; PN CL03A224MQ3NNNC -> (none)
- C11, C8: MPN (none) -> GRM155R60J106ME44D; PN GRM155R60J106ME15D -> (none)
- C12, C46, C47: MPN (none) -> GRM155R61A475MEAAD; PN GRM155R61A475MEAAD -> (none)
- C14, C2, C5: MPN (none) -> GRM033R61C103KA12D; PN GRM033R61C103KA12D -> (none)
- C15, C16, C6, C83, C9: MPN (none) -> CL03A104KQ3NNNC; PN CL03A104KQ3NNNC -> (none)
- C17, C18, C7: Info (none) -> 6.3V, X5R; MPN (none) -> GRM155R60J106ME44D; PN GRM155R60J106ME15D -> (none)
- C3: MPN (none) -> LMK107BBJ106MALT; PN LMK107BBJ106MALT -> (none)
- R1, R13, R14, R25: MPN (none) -> RC0201FR-07100KL; PN RC0201FR-07100KL -> (none)
- R15: value 120K -> 120K 1%; footprint Resistor_SMD:R_0201_0603Metric -> Resistor_SMD:R_0402_1005Metric
- R16: value 82K -> 82K 1%; footprint Resistor_SMD:R_0201_0603Metric -> Resistor_SMD:R_0402_1005Metric
- R17, R18, R5: value 100k -> 100k 1%; MPN (none) -> RC0201FR-07100KL; PN RC0201FR-07100KL -> (none)
- R2: value 22K -> 22K 1%; footprint Resistor_SMD:R_0201_0603Metric -> Resistor_SMD:R_0402_1005Metric
- R6: MPN (none) -> RC0402FR-070RL; PN RC0402FR-070RL -> (none)
- U1: MPN (none) -> EA3036CQBR; PN EA3036CQBR -> (none)
- U8: MPN (none) -> TPS51206DSQR; PN TPS51206DSQR -> (none)
Connections:
- net GND: now also C11.2, C17.2, C18.2, C7.2, C28.2, R34.1, U2.2 (GND), U7.2 (GND), U7.5 (GND); no longer C11.1, C17.1, C18.1, C7.1
- net P1.1V: now also C17.1; no longer C17.2
- net P1.35V: now also C18.1; no longer C18.2
- net P2.5V: now also JP2.2 (C); no longer C47.1
- net P3.3V: now also C7.1, D2.2 (A), JP1.3 (B), U2.3 (VIN), U7.4 (IN); no longer C7.2
- net PGOOD_P1.1V: now also U2.5 (EN), U7.3 (EN)
- net PUSB_VBUS: now also JP1.1 (A); no longer C14.2, C2.2, C3.2, C5.2, U1.16 (VCC), U1.19 (VIN3), U1.7 (VIN2)
- net VTT: now also C11.1; no longer C11.2
- new net: C13.2, C47.1, JP2.3 (B), L4.1, R33.1
- new net: C13.1, R33.2, R34.2, U2.1 (FB)
- new net: L4.2, U2.4 (SW)
- new net: C28.1, JP2.1 (A), U7.1 (OUT)
- new net VSYS: C14.2, C2.2, C3.2, C5.2, D2.1 (K), JP1.2 (C), U1.16 (VCC), U1.19 (VIN3), U1.7 (VIN2)
Other:
- note added: "Suggested upgrade 5V to 3V with othe chip 2.5V with part of the current chip"
- note added: "ULX3S"
- note added: "Vth=1.2V"
- note added: "soldiercrab TLV62569ADRLR"
- company: (none) -> (C) 2023-2026 Victor Suarez Rovere
- title: (none) -> FPGA board
- moved on the sheet: C46, C47, R25
