File: hardware/FPGA_board/fileSDMMC.kicad_sch (KiCad schematic)
At the start: 6 parts, among them J4 MicroSd

Commit message: update PCB design files
Parts:
- removed J4: MicroSd, Connector_Card:microSD_HC_Molex_104031-0811, symbol Connector_Generic_MountingPin:Conn_01x09_MountingPin
- added C29: 100nF, Capacitor_SMD:C_0201_0603Metric, symbol Device:C
- added J9: TF TF-018 1.5mm, Library:TF-SMD_TF-018, symbol TF 1.5H 短体
- added JP3: SolderJumper_2_Open, Jumper:SolderJumper-2_P1.3mm_Open_RoundedPad1.0x1.5mm, symbol Jumper:SolderJumper_2_Open
- added R35, R36, R38, R39: 15, Resistor_SMD:R_0201_0603Metric, symbol Device:R
- added R37: 75, Resistor_SMD:R_0201_0603Metric, symbol Device:R
- added TP3, TP4: SMD_TP, TestPoint:TestPoint_Pad_D1.0mm, symbol Connector:TestPoint_Flag
- added U5: Si5351A-B-GT, Package_SO:MSOP-10_3x3mm_P0.5mm, symbol Oscillator:Si5351A-B-GT
- added Y1: 27MHz, Crystal:Crystal_SMD_2016-4Pin_2.0x1.6mm, symbol Device:Crystal_GND24_Small
- C70: MPN (none) -> CL03A104KQ3NNNC; PN CL03A104KQ3NNNC -> (none)
- C71: MPN (none) -> CL10A475KP8NNNC; PN CL10A475KP8NNNC -> (none)
- FB1: MPN (none) -> BLM15AG601SN1D; PN BLM15AG601SN1D -> (none)
- R28: Mfg ‎Yageo‎ -> (none); PN RC0201FR-0710KL -> (none)
- RN7: MPN (none) -> 4D02WGJ0103TCE; Mfg YAGEO -> (none); PN YC124-JR-0710KL -> (none)
Connections:
- net GND: now also C29.1, J9.10 (GND), J9.6 (VSS), U5.8 (GND), Y1.2, Y1.4
- net P3.3V: now also C29.2, U5.1 (VDD); no longer R28.1, RN7.5 (R4.2), RN7.6 (R3.2), RN7.7 (R2.2), RN7.8 (R1.2)
- net SD0_CD: now also J9.9 (CD)
- net SD0_CLK: now also J9.5 (CLK)
- net SD0_CMD: now also RN7.2 (R2.1), J9.3 (CMD); no longer RN7.3 (R3.1)
- net SD0_DAT0: now also RN7.3 (R3.1), J9.7 (DATA0); no longer RN7.2 (R2.1)
- net SD0_DAT1: now also RN7.4 (R4.1), J9.8 (DATA1); no longer RN7.1 (R1.1)
- net SD0_DAT2: now also RN7.1 (R1.1), J9.1 (DATA2); no longer RN7.4 (R4.1)
- net SD0_DAT3: now also J9.2 (CD/DATA3)
- net VDD_SD: now reaches C70.2, C71.1, FB1.1
- net VDD_SD: now also R28.1, RN7.5 (R4.2), RN7.6 (R3.2), RN7.7 (R2.2), RN7.8 (R1.2), J9.4 (VDD)
- new net: R35.1, R37.1, R38.2
- new net: R36.1, R37.2, R39.2
- new net: JP3.1 (A), U5.6 (CLK2)
- new net: R35.2, U5.10 (CLK0)
- new net: R36.2, U5.9 (CLK1)
- new net: U5.3 (XB), Y1.1
- new net: U5.2 (XA), Y1.3
- new net EXT_PLL+: R38.1, TP3.1
- new net EXT_PLL-: R39.1, TP4.1
- new net IO_SCL: U5.5 (SDA)
- new net IO_SDA: U5.4 (SCL)
- new net LED_B: JP3.2 (B)
- new net P2.5V: U5.7 (VDDO)
Other:
- note removed: "DAT2 DAT3/CD CMD VDD CLK VSS DAT0 DAT1 DET"
- company: (none) -> (C) 2023-2026 Victor Suarez Rovere
- title: (none) -> FPGA board

Commit message: Add documentation regarding DFM analysis and corresponding changes to the 6-layer board design
Parts:
- Y1: LCSC Part Number (none) -> C18214311
Changed lines of the file:
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@@
+			)
+		)
+		(property "LCSC Part Number" "C18214311"
+			(at 82.55 154.94 90)
+			(effects
+				(font
+					(size 1.27 1.27)
+				)
+				(hide yes)
 			)
 		)
