File: hardware/LVDS_adapter/LVDS_adapter.kicad_pcb (KiCad board)
At the start: 2 copper layers, 47 x 31 mm, 12 parts, among them J1 DF12NB(3.0)-30DS-0.5V(51), J2 LVDS, J3 BAKLIGHT_POWER

Commit message: update PCB design files
Parts:
- removed the G*** at (185.6, 106.9)
- moved TP2 4.21 mm to (183.9, 97.7)
- moved TP1 3.79 mm to (184.3, 93.3)
Other:
- board text added: "CERN OHL-S license"
- board text added: "NORTH"
- board text removed: "CERN OHL-S License"
