File: hardware/LVDS_adapter/LVDS_adapter_(2ch-8bit).kicad_sch (KiCad schematic)
At the start: 15 parts, among them J1 DF12NB(3.0)-30DS-0.5V(51), J2 Conn_02x15_Odd_Even, J3 Conn_01x06_Socket, J4 DF12NB(3.0)-30DS-0.5V(51), J5 Conn_01x06_Socket, J6 Conn_01x02

Commit message: change 2x15 vertical header for an edge one
Changed lines of the file:
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@@
 	)
 	(junction
+		(at 178.435 112.395)
+		(diameter 0)
+		(color 0 0 0 0)
+	)
+	(junction
 		(at 121.92 104.775)
 		(diameter 0)
@@
 	)
 	(junction
-		(at 178.435 112.395)
-		(diameter 0)
-		(color 0 0 0 0)
-	)
-	(junction
 		(at 121.92 125.095)
 		(diameter 0)
@@
 	(wire
 		(pts
-			(xy 172.085 112.395) (xy 178.435 112.395)
-		)
-		(stroke
-			(width 0)
-			(type default)
-		)
-	)
-	(wire
-		(pts
 			(xy 101.6 81.915) (xy 121.92 81.915)
 		)
@@
 	(wire
 		(pts
-			(xy 178.435 112.395) (xy 191.135 112.395)
+			(xy 172.085 112.395) (xy 178.435 112.395)
 		)
 		(stroke
@@
 	(wire
 		(pts
+			(xy 178.435 112.395) (xy 191.135 112.395)
+		)
+		(stroke
+			(width 0)
+			(type default)
+		)
+	)
+	(wire
+		(pts
 			(xy 121.92 122.555) (xy 135.255 122.555)
 		)
@@
 				)
 				(justify left)
+				(hide yes)
 			)
 		)
