File: hardware/eDP_adapter/eDP_adapter.kicad_pcb (KiCad board)
At the start: 2 copper layers, 36.1 x 28.4 mm, 87 parts, among them J1 DF12NB(3.0)-30DS-0.5V(51), J2 DF12NB(3.0)-30DS-0.5V(51), J3 Conn_01x40, J4 Barrel_Jack_MountingPin, Q1 2N7002WT1G, U1 NCS8801, U2 EA3036A, U3 MT3608

Commit message: update PCB design files
Parts:
- added G***: LOGO, LOGO, B.Cu at (109.0, 133.3)
- added G***: LOGO, LOGO, B.Cu at (123.1, 133.2)
Routing:
- net +3V3_MCU: track 1.15 -> 0.45 mm
- net B1: track 20.4 -> 21.0 mm
- net GND: vias 37 -> 38
Other:
- board size 36.1 x 28.4 mm -> 36.3 x 28.4 mm
