File: hardware/eDP_adapter/eDP_adapter.kicad_sch (KiCad schematic)
At the start: 90 parts, among them J1 DF12NB(3.0)-30DS-0.5V(51), J2 DF12NB(3.0)-30DS-0.5V(51), J3 Conn_01x40, J4 Barrel_Jack_MountingPin, Q1 2N7002WT1G, U1 NCS8801, U2 EA3036A, U3 MT3608

Commit message: update PCB design files
Parts:
- R9: LCSC Part Number C25940 -> (none)
Changed lines of the file:
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@@
 			)
 		)
-		(property "LCSC Part Number" "C25940"
+		(property "LCSC Part Number" ""
 			(at 22.86 167.64 0)
 			(effects
