File: hardware/eDP_adapter/eDP_adapter_power.kicad_sch (KiCad schematic)
At the start: 43 parts, among them J4 Barrel_Jack_MountingPin, Q1 NX3008NBKW,115, U2 TLV62569APDRL, U3 MT3608, U5 TPNCP115ASN120T2G

Commit message: change eDP adapter for dual channel LVDS input mode
Parts:
- U5: MPN_ALT (none) -> AP2112K-1.2TRG1
Other:
- note removed: "The IC may require a higher voltage"
Changed lines of the file:
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@@
 		)
 	)
-	(text "The IC may require a higher voltage"
-		(exclude_from_sim no)
-		(at 69.088 184.15 0)
-		(effects
-			(font
-				(size 2 2)
-				(thickness 0.4)
-				(bold yes)
-			)
-		)
-	)
 	(global_label "XVDD_3V3"
 		(shape input)
@@
 			(at 64.135 162.56 0)
 			(effects
+				(font
+					(size 1.27 1.27)
+				)
+				(hide yes)
+			)
+		)
+		(property "MPN_ALT" "AP2112K-1.2TRG1"
+			(at 64.135 162.56 0)
+			(effects
