File: hardware/eDP_adapter/eDP_adapter_IORGB.kicad_sch (KiCad schematic)
At the start: 12 parts, among them J1 DF12NB(3.0)-30DS-0.5V(51), J2 DF12NB(3.0)-30DS-0.5V(51), J3 Conn_01x30, J5 Conn_01x06_Socket

Commit message: move 6-pin I2C FPC connector to bottom, and add missing schematics subsheets
Parts:
- removed TP1, TP2: TestPoint_Small, TestPoint:TestPoint_Pad_D1.0mm, symbol Connector:TestPoint_Small
- added TP10, TP11, TP12, TP13, TP14: TestPoint_Small, TestPoint:TestPoint_Pad_D1.0mm, symbol Connector:TestPoint_Small
Connections:
- net SCK: now also TP14.1; no longer J3.24 (Pin_24)
- net SDA: now also TP13.1; no longer J3.25 (Pin_25)
- net TP_INT: no longer J3.14 (Pin_14), TP7.1
- net LCD_HSYNC: now reaches J1.10 (9)
- net LCD_HSYNC: now also TP11.1
- net LCD_VSYNC: now reaches J1.12 (11)
- net LCD_VSYNC: now also TP12.1
- net G1: now reaches J1.14 (13)
- net B1: now reaches J1.2 (1)
- net G0: now reaches J1.20 (19)
- net B0: now reaches J1.8 (7)
- net R1: now reaches J2.27 (28)
- net R0: now reaches J2.29 (30)
- net E0+ renamed G6
- net E0- renamed G7
- net E1+ renamed R2
- net E1- renamed R3
- net E2+ renamed R4
- net E2- renamed R5
- net E3+ renamed PCLK
- net E3- renamed LCD_DE
- net LCD_DE: now also TP10.1
- net EC+ renamed R6
- net EC- renamed R7
- net O0+ renamed B2
- net O0- renamed B3
- net O1+ renamed B4
- net O1- renamed B5
- net O2+ renamed B6
- net O2- renamed B7
- net O3+ renamed G4
- net O3- renamed G5
- net OC+ renamed G2
- net OC- renamed G3
- new net LCD_TEST: J3.14 (Pin_14), TP7.1
- no-connect marks 20 -> 23
Other:
- note added: "LCD_D0"
- note added: "LCD_D1"
- note added: "LCD_D10"
- note added: "LCD_D11"
- note added: "LCD_D12"
- note added: "LCD_D13"
- note added: "LCD_D14"
- note added: "LCD_D15"
- note added: "LCD_D16"
- note added: "LCD_D17"
- note added: "LCD_D18"
- note added: "LCD_D19"
- note added: "LCD_D2"
- note added: "LCD_D20"
- note added: "LCD_D21"
- note added: "LCD_D22"
- note added: "LCD_D23"
- note added: "LCD_D3"
- note added: "LCD_D4"
- note added: "LCD_D5"
- note added: "LCD_D7"
- note added: "LCD_D8"
- note added: "LCD_D9"
