File: hardware/eDP_adapter/eDP_adapter_IO.kicad_sch (KiCad schematic)
At the start: 12 parts, among them J1 DF12NB(3.0)-30DS-0.5V(51), J2 DF12NB(3.0)-30DS-0.5V(51), J3 Conn_01x30, J5 Conn_01x06_Socket

Commit message: change 6-pin I2C connector to one with top contacts
Parts:
- removed J3: Conn_01x30, easyeda2kicad:FPC-SMD_30P-P0.50_FPC-0.5FX-30PWBH15, symbol Connector_Generic:Conn_01x30
- removed J5: Conn_01x06_Socket, easyeda2kicad:FPC-SMD_FH52K-6S-0.5SH, symbol Connector:Conn_01x06_Socket
- added J3: Conn_01x30, easyeda2kicad:FPC-SMD_30P-P0.50_FPC-0.5FX-30PWBH15, symbol Connector_Generic_MountingPin:Conn_01x30_MountingPin
- added J5: Conn_01x06_Socket, easyeda2kicad:CONN-SMD_527450697, symbol Connector_Generic_MountingPin:Conn_01x06_MountingPin
Connections:
- net +3V3: now also J5.2 (Pin_2)
- net +3V3_DISP: now also J3.12 (Pin_12), J3.13 (Pin_13)
- net AUX0_N: now also J3.10 (Pin_10)
- net AUX0_P: now also J3.9 (Pin_9)
- net BACKLIGHT_POWER: now also J3.26 (Pin_26), J3.27 (Pin_27), J3.28 (Pin_28), J3.29 (Pin_29)
- net GND: now also J3.11 (Pin_11), J3.15 (Pin_15), J3.16 (Pin_16), J3.18 (Pin_18), J3.19 (Pin_19), J3.2 (Pin_2), J3.20 (Pin_20), J3.21 (Pin_21), J3.5 (Pin_5), J3.8 (Pin_8), J3.MP (MountPin), J5.3 (Pin_3), J5.MP (MountPin)
- net HPD: now also J3.17 (Pin_17)
- net LCD_PWM: now also J3.23 (Pin_23)
- net PSEL: now also J3.22 (Pin_22), J5.1 (Pin_1)
- net SCK: now also J3.24 (Pin_24), J5.6 (Pin_6)
- net SDA: now also J3.25 (Pin_25), J5.5 (Pin_5)
- net TP_INT: now also J3.14 (Pin_14), J5.4 (Pin_4)
- net TX0_N: now also J3.6 (Pin_6)
- net TX0_P: now also J3.7 (Pin_7)
- net TX1_N: now also J3.3 (Pin_3)
- net TX1_P: now also J3.4 (Pin_4)
