File: hardware/IO_board/IO_board.kicad_sch (KiCad schematic)
At the start: 7 parts, among them J1 DF12NB(3.0)-30DS-0.5V(51), J2 Combined I/O, J3 Conn_01x31, J4 DF12NB(3.0)-30DS-0.5V(51), J5 Conn_01x31, J6 Conn_01x06, J7 Combined I/O

Commit message: fixed mixup of pins G5/G4 (3rd diff pair ODD) and DE/PCLK (3rd diff pair EVEN), now with correct polarity for diff pairs
Connections:
- net G4: now also J4.6 (5); no longer J4.4 (3)
- net G5: now also J4.4 (3); no longer J4.6 (5)
Other:
- note added: "LVDS0-V3N LCD0-D13 LVDS0-V3P LCD0-D12"
- note removed: "LVDS0-V3P LCD0-D12 LVDS0-V3N LCD0-D13"
Changed lines of the file:
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@@
 		)
 	)
-	(text "LVDS0-V3P LCD0-D12 \nLVDS0-V3N LCD0-D13 \n"
+	(text "LVDS0-V3N LCD0-D13 \nLVDS0-V3P LCD0-D12 \n"
 		(exclude_from_sim no)
 		(at 46.99 140.716 0)
@@
 		)
 	)
+	(label "G5"
+		(at 62.23 139.7 0)
+		(fields_autoplaced yes)
+		(effects
+			(font
+				(size 1.27 1.27)
+			)
+			(justify left bottom)
+		)
+	)
 	(label "G1"
 		(at 59.69 57.15 180)
@@
 		)
 	)
-	(label "G4"
-		(at 64.77 139.7 0)
-		(fields_autoplaced yes)
-		(effects
-			(font
-				(size 1.27 1.27)
-			)
-			(justify left bottom)
-		)
-	)
 	(label "VIO"
 		(at 148.59 93.98 0)
@@
 		)
 	)
+	(label "G4"
+		(at 62.23 142.24 0)
+		(fields_autoplaced yes)
+		(effects
+			(font
+				(size 1.27 1.27)
+			)
+			(justify left bottom)
+		)
+	)
 	(label "SCL"
 		(at 148.59 81.28 0)
@@
 		)
 	)
-	(label "G5"
-		(at 64.77 142.24 0)
-		(fields_autoplaced yes)
-		(effects
-			(font
-				(size 1.27 1.27)
-			)
-			(justify left bottom)
-		)
-	)
