File: hardware/eDP_adapter/edp_adapterITE/eDP_adapter_IO.kicad_sch (KiCad schematic)
At the start: 12 parts, among them J1 DF12NB(3.0)-30DS-0.5V(51), J2 DF12NB(3.0)-30DS-0.5V(51), J3 Conn_01x30, J5 Conn_01x06_Socket

Commit message: change 6-pin I2C connector to one with top contacts
Parts:
- J3: symbol Connector_Generic:Conn_01x30 -> Connector_Generic_MountingPin:Conn_01x30_MountingPin
- J5: footprint easyeda2kicad:FPC-SMD_FH52K-6S-0.5SH -> easyeda2kicad:CONN-SMD_527450697; symbol Connector:Conn_01x06_Socket -> Connector_Generic_MountingPin:Conn_01x06_MountingPin; MFG (none) -> Molex; MPN FH52K-6S-0.5SH -> 527450697
Connections:
- net GND: now also J3.MP (MountPin), J5.MP (MountPin)
Other:
- moved on the sheet: J5
Changed lines of the file:
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@@
 	(wire
 		(pts
+			(xy 217.17 73.025) (xy 217.17 71.755)
+		)
+		(stroke
+			(width 0)
+			(type default)
+		)
+	)
+	(wire
+		(pts
 			(xy 62.865 79.375) (xy 65.405 79.375)
 		)
@@
 	(wire
 		(pts
+			(xy 224.79 71.755) (xy 224.79 73.66)
+		)
+		(stroke
+			(width 0)
+			(type default)
+		)
+	)
+	(wire
+		(pts
 			(xy 64.135 69.215) (xy 67.945 69.215)
 		)
@@
 	(wire
 		(pts
+			(xy 217.17 71.755) (xy 224.79 71.755)
+		)
+		(stroke
+			(width 0)
+			(type default)
+		)
+	)
+	(wire
+		(pts
 			(xy 67.945 76.835) (xy 52.705 76.835)
 		)
@@
 	(symbol
 		(lib_id "power:GND")
+		(at 217.17 73.025 0)
+		(mirror y)
+		(unit 1)
+		(exclude_from_sim no)
+		(in_bom yes)
+		(on_board yes)
+		(dnp no)
+		(property "Reference" "#PWR059"
+			(at 217.17 79.375 0)
+			(effects
+				(font
+					(size 1.27 1.27)
+				)
+				(hide yes)
+			)
+		)
+		(property "Value" "GND"
+			(at 212.852 74.676 0)
+			(effects
+				(font
+					(size 1.27 1.27)
+				)
+			)
+		)
+		(property "Footprint" ""
+			(at 217.17 73.025 0)
+			(effects
+				(font
+					(size 1.27 1.27)
+				)
+				(hide yes)
+			)
+		)
+		(property "Datasheet" ""
+			(at 217.17 73.025 0)
+			(effects
+				(font
+					(size 1.27 1.27)
+				)
+				(hide yes)
+			)
+		)
+		(property "Description" "Power symbol creates a global label with name \"GND\" , ground"
+			(at 217.17 73.025 0)
+			(effects
+				(font
+					(size 1.27 1.27)
+				)
+				(hide yes)
+			)
+		)
+		(pin "1"
+		)
+		(instances
+			(project "edp_adapterITE"
+				(path "/971d21cc-a5c8-4932-ad62-f68d6b0e4b00/5642edec-fdb1-4594-a460-4c5875e7b593"
+					(reference "#PWR059")
+					(unit 1)
+				)
+			)
+		)
+	)
+	(symbol
+		(lib_id "power:GND")
 		(at 217.17 46.355 0)
 		(mirror y)
@@
 	)
 	(symbol
-		(lib_id "Connector_Generic:Conn_01x30")
+		(lib_id "power:GND")
+		(at 222.885 59.055 0)
+		(mirror y)
+		(unit 1)
+		(exclude_from_sim no)
+		(in_bom yes)
+		(on_board yes)
+		(dnp no)
+		(property "Reference" "#PWR048"
+			(at 222.885 65.405 0)
+			(effects
+				(font
+					(size 1.27 1.27)
+				)
+				(hide yes)
+			)
+		)
+		(property "Value" "GND"
+			(at 218.567 60.706 0)
+			(effects
+				(font
+					(size 1.27 1.27)
+				)
+			)
+		)
+		(property "Footprint" ""
+			(at 222.885 59.055 0)
+			(effects
+				(font
+					(size 1.27 1.27)
+				)
+				(hide yes)
+			)
+		)
+		(property "Datasheet" ""
+			(at 222.885 59.055 0)
+			(effects
+				(font
+					(size 1.27 1.27)
+				)
+				(hide yes)
+			)
+		)
+		(property "Description" "Power symbol creates a global label with name \"GND\" , ground"
+			(at 222.885 59.055 0)
+			(effects
+				(font
+					(size 1.27 1.27)
+				)
+				(hide yes)
+			)
+		)
+		(pin "1"
+		)
+		(instances
+			(project "edp_adapterITE"
+				(path "/971d21cc-a5c8-4932-ad62-f68d6b0e4b00/5642edec-fdb1-4594-a460-4c5875e7b593"
+					(reference "#PWR048")
+					(unit 1)
+				)
+			)
+		)
+	)
+	(symbol
+		(lib_id "Connector_Generic_MountingPin:Conn_01x30_MountingPin")
 		(at 224.79 116.84 0)
 		(mirror x)
@@
 			)
 		)
-		(property "Description" "Generic connector, single row, 01x30, script generated (kicad-library-utils/schlib/autogen/connector/)"
+		(property "Description" "Generic connectable mounting pin connector, single row, 01x30, script generated (kicad-library-utils/schlib/autogen/connector/)"
 			(at 224.79 116.84 0)
 			(effects
@@
 		(pin "9"
 		)
+		(pin "MP"
+		)
 		(instances
 			(project "edp_adapterITE"
@@
 	)
 	(symbol
-		(lib_id "Connector:Conn_01x06_Socket")
+		(lib_id "Connector_Generic_MountingPin:Conn_01x06_MountingPin")
 		(at 222.885 46.355 0)
 		(unit 1)
@@
 			)
 		)
-		(property "Footprint" "easyeda2kicad:FPC-SMD_FH52K-6S-0.5SH"
+		(property "Footprint" "easyeda2kicad:CONN-SMD_527450697"
 			(at 222.885 46.355 0)
 			(effects
@@
 			)
 		)
-		(property "Description" "Generic connector, single row, 01x06, script generated"
+		(property "Description" "Generic connectable mounting pin connector, single row, 01x06, script generated (kicad-library-utils/schlib/autogen/connector/)"
 			(at 222.885 46.355 0)
 			(effects
@@
 			)
 		)
-		(property "MPN" "FH52K-6S-0.5SH"
+		(property "MPN" "527450697"
+			(at 222.885 46.355 0)
+			(effects
+				(font
+					(size 1.27 1.27)
+				)
+				(hide yes)
+			)
+		)
+		(property "MFG" "Molex"
 			(at 222.885 46.355 0)
 			(effects
@@
 		(pin "6"
 		)
+		(pin "MP"
+		)
 		(instances
