File: hardware/eDP_adapter/edp_adapterITE/edp_adapterITE.kicad_sch (KiCad schematic)
At the start: 39 parts, among them U4 IT6251, X1 27MHz

Commit message: add output serpentines to eDP adapter "B" board
Parts:
- removed C10, C13, C18, C20, C21, C27, C28, C29, C3, C30, C31, C33, C34, C35, C36, C5, C7, C8: 0.1uF, Library:C_0402_1005Metric, symbol Periph-altium-import:0_CAP
- removed R18: 1M, Resistor_SMD:R_0402_1005Metric, symbol Device:R
- added R3: 1M, Resistor_SMD:R_0402_1005Metric, symbol Device:R
Connections:
- net XTALI: now also R3.2
- net XTALO: now also R3.1
Other:
- note added: "inter skew is possible in eDP intra skew is not"
- note removed: "skew < 50mil"
- title: eDP Adapter board ITE -> (none)
- moved on the sheet: C1, C14, C15, C16, C17, C23, C32, C37, CR1, CR2, CR3, R1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

Commit message: update part numbers for manufacturing
Parts:
- U4: LCSC Part C9900011361 -> (none); LCSC Part Number (none) -> C9900011361
Changed lines of the file:
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@@
 			)
 		)
-		(property "LCSC Part" "C9900011361"
+		(property "LCSC Part Number" "C9900011361"
 			(at 73.025 97.79 0)
 			(effects
