File: hardware/eDP_adapter/edp_adapterITE/eDP_adapter_power.kicad_sch (KiCad schematic)
At the start: 48 parts, among them J4 Barrel_Jack_MountingPin, U1 AMS1117-1.8, U2 TLV62569APDRL, U3 MT3608

Commit message: update part numbers for manufacturing
Parts:
- U1: LCSC Part Number (none) -> C347220
Changed lines of the file:
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@@
+			)
+		)
+		(property "LCSC Part Number" "C347220"
+			(at 139.7 50.8 0)
+			(effects
+				(font
+					(size 1.27 1.27)
+				)
+				(hide yes)
 			)
 		)

Commit message: fixes for producion and notes
Parts:
- C6: MPN GRM033R61C103KA12D -> (none)
Changed lines of the file:
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@@
-			)
-		)
-		(property "MPN" "GRM033R61C103KA12D"
-			(at 63.5 101.6 0)
-			(effects
-				(font
-					(size 1.27 1.27)
-				)
-				(hide yes)
 			)
 		)
