File: hardware/Spartan6_board/fpga_ddr.kicad_sch (KiCad schematic)
At the start: 37 parts, among them U12 MT41K64M16TW, U5 XC6SLX16-FTG256

Commit message: change DVI FPC pinout to match DVI connector (G-S-S-G), and FPGA device from XC6SLX16-FTG256 to XC6SLX25-3FTG256C
Parts:
- U5: value XC6SLX16-FTG256 -> XC6SLX25-3FTG256C; LCSC Part Number C39313 -> C1521716
Other:
- note added: "Consider the slower MT46H32M16LF (8x9mm) as in Saturn board"
- title: Caster EPDC -> Spartan 6 FPGA board
Changed lines of the file:
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@@
 	(paper "A4")
 	(title_block
-		(title "Caster EPDC")
-		(date "2022-07-03")
-		(rev "R0.4")
+		(title "Spartan 6 FPGA board")
+		(date "2026-09-17")
+		(rev "R0.1")
 		(company "Copyright 2022 Modos / Engineer: Wenting Zhang")
 	)
@@
 		)
 	)
+	(text "Consider the slower MT46H32M16LF (8x9mm)\nas in Saturn board"
+		(exclude_from_sim no)
+		(at 258.064 18.288 0)
+		(effects
+			(font
+				(size 1.27 1.27)
+			)
+		)
+	)
 	(text "ZIO"
 		(exclude_from_sim no)
@@
 			)
 		)
-		(property "Value" "XC6SLX16-FTG256"
+		(property "Value" "XC6SLX25-3FTG256C"
 			(at 86.36 187.96 0)
 			(effects
@@
 			)
 		)
-		(property "LCSC Part Number" "C39313"
+		(property "LCSC Part Number" "C1521716"
 			(at 86.36 104.14 0)
 			(effects

Commit message: review and update manufacturing constraints (via size, etc.)
Other:
- company: Copyright 2022 Modos / Engineer: Wenting Zhang -> (C) 2025-2026 Victor Suarez Rovere <suarezvictor@gmail.com>
Changed lines of the file:
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@@
 	(title_block
 		(title "Spartan 6 FPGA board")
-		(date "2026-09-17")
+		(date "2026-09-18")
 		(rev "R0.1")
-		(company "Copyright 2022 Modos / Engineer: Wenting Zhang")
+		(company "(C) 2025-2026 Victor Suarez Rovere <suarezvictor@gmail.com>")
+		(comment 1 "Copyright 2023 Modos / Engineer: Wenting Zhang")
 	)
 	(junction
