File: hardware/Spartan6_board/mcu.kicad_sch (KiCad schematic)
At the start: 29 parts, among them J1 USB_C_Receptacle_USB2.0, J5 SWD, SW1 TS-1007S-AR02516, SW2 TS-1007S-AR02516, U13 W25Q32JV, U14 RP2040, U15 USBLC6-2P6, Y2 12MHz

Commit message: change DVI FPC pinout to match DVI connector (G-S-S-G), and FPGA device from XC6SLX16-FTG256 to XC6SLX25-3FTG256C
Other:
- title: Caster EPDC -> Spartan 6 FPGA board
Changed lines of the file:
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@@
 	(paper "A4")
 	(title_block
-		(title "Caster EPDC")
-		(date "2022-07-03")
-		(rev "R0.4")
+		(title "Spartan 6 FPGA board")
+		(date "2026-09-17")
+		(rev "R0.1")
 		(company "Copyright 2022 Modos / Engineer: Wenting Zhang")
 	)

Commit message: review and update manufacturing constraints (via size, etc.)
Parts:
- added TP14, TP15, TP16, TP17: TestPoint_Small, TestPoint:TestPoint_Pad_D1.5mm, symbol Connector:TestPoint_Small
Connections:
- net GPIO5 is gone; now on net DDC_SDA: U14.7 (GPIO5)
- net GPIO6 is gone; now on net DDC_SCL: U14.8 (GPIO6)
- net GPIO7 is gone; now on net KEY: U14.9 (GPIO7)
- net DDC_SCL: no longer U14.3 (GPIO1)
- net DDC_SDA: no longer U14.2 (GPIO0)
- net GPIO3: now also TP17.1
- net KEY: no longer U14.4 (GPIO2)
- new net GPIO0: TP14.1, U14.2 (GPIO0)
- new net GPIO1: TP15.1, U14.3 (GPIO1)
- new net GPIO2: TP16.1, U14.4 (GPIO2)
Other:
- company: Copyright 2022 Modos / Engineer: Wenting Zhang -> (C) 2025-2026 Victor Suarez Rovere <suarezvictor@gmail.com>

Commit message: fix R0/R1 mixup
Changed lines of the file:
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@@
 (kicad_sch
-	(version 20231120)
+	(version 20250114)
 	(generator "eeschema")
-	(generator_version "8.0")
+	(generator_version "9.0")
 	(paper "A4")
 	(title_block
@@
 	(label "XIN"
 		(at 121.92 127 180)
-		(fields_autoplaced yes)
 		(effects
 			(font
@@
 	(label "QSPI_SD2"
 		(at 119.38 109.22 180)
-		(fields_autoplaced yes)
 		(effects
 			(font
@@
 	(label "QSPI_SD0"
 		(at 154.94 86.36 0)
-		(fields_autoplaced yes)
 		(effects
 			(font
@@
 	(label "GPIO4"
 		(at 233.68 73.66 180)
-		(fields_autoplaced yes)
 		(effects
 			(font
@@
 	(label "QSPI_SD3"
 		(at 119.38 111.76 180)
-		(fields_autoplaced yes)
 		(effects
 			(font
@@
 	(label "XOUT"
 		(at 121.92 139.7 180)
-		(fields_autoplaced yes)
 		(effects
 			(font
@@
 	(label "GPIO27_ADC1"
 		(at 233.68 134.62 180)
-		(fields_autoplaced yes)
 		(effects
 			(font
@@
 	(label "GPIO13"
 		(at 233.68 96.52 180)
-		(fields_autoplaced yes)
 		(effects
 			(font
@@
 	(label "QSPI_SD0"
 		(at 119.38 101.6 180)
-		(fields_autoplaced yes)
 		(effects
 			(font
@@
 	(label "USB_DN"
 		(at 142.24 73.66 0)
-		(fields_autoplaced yes)
 		(effects
 			(font
@@
 	(label "GPIO23"
 		(at 233.68 121.92 180)
-		(fields_autoplaced yes)
 		(effects
 			(font
@@
 	(label "QSPI_SS"
 		(at 73.66 104.14 0)
-		(fields_autoplaced yes)
 		(effects
 			(font
@@
 	(label "GPIO11"
 		(at 233.68 91.44 180)
-		(fields_autoplaced yes)
 		(effects
 			(font
@@
 	(label "GPIO20"
 		(at 233.68 114.3 180)
-		(fields_autoplaced yes)
 		(effects
 			(font
@@
 	(label "XIN"
 		(at 154.94 109.22 0)
-		(fields_autoplaced yes)
 		(effects
 			(font
@@
 	(label "GPIO14"
 		(at 233.68 99.06 180)
-		(fields_autoplaced yes)
 		(effects
 			(font
@@
 	(label "QSPI_SD1"
 		(at 154.94 88.9 0)
-		(fields_autoplaced yes)
 		(effects
 			(font
@@
 	(label "GPIO5"
 		(at 233.68 76.2 180)
-		(fields_autoplaced yes)
 		(effects
 			(font
@@
 	(label "GPIO16"
 		(at 233.68 104.14 180)
-		(fields_autoplaced yes)
 		(effects
 			(font
@@
 	(label "GPIO26_ADC0"
 		(at 233.68 132.08 180)
-		(fields_autoplaced yes)
 		(effects
 			(font
@@
 	(label "GPIO0"
 		(at 233.68 63.5 180)
-		(fields_autoplaced yes)
 		(effects
 			(font
@@
 	(label "GPIO9"
 		(at 233.68 86.36 180)
-		(fields_autoplaced yes)
 		(effects
 			(font
@@
 	(label "GPIO7"
 		(at 233.68 81.28 180)
-		(fields_autoplaced yes)
 		(effects
 			(font
@@
 	(label "XOUT"
 		(at 154.94 119.38 0)
-		(fields_autoplaced yes)
 		(effects
 			(font
@@
 	(label "QSPI_SCLK"
 		(at 73.66 109.22 0)
-		(fields_autoplaced yes)
 		(effects
 			(font
@@
 	(label "GPIO21"
 		(at 233.68 116.84 180)
-		(fields_autoplaced yes)
 		(effects
 			(font
@@
 	(label "GPIO22"
 		(at 233.68 119.38 180)
-		(fields_autoplaced yes)
 		(effects
 			(font
@@
 	(label "QSPI_SD1"
 		(at 119.38 104.14 180)
-		(fields_autoplaced yes)
 		(effects
 			(font
@@
 	(label "SWCLK"
 		(at 154.94 129.54 0)
-		(fields_autoplaced yes)
 		(effects
 			(font
@@
 	(label "GPIO18"
 		(at 233.68 109.22 180)
-		(fields_autoplaced yes)
 		(effects
 			(font
@@
 	(label "GPIO6"
 		(at 233.68 78.74 180)
-		(fields_autoplaced yes)
 		(effects
 			(font
@@
 	(label "SWD"
 		(at 154.94 132.08 0)
-		(fields_autoplaced yes)
 		(effects
 			(font
@@
 	(label "RUN"
 		(at 154.94 63.5 0)
-		(fields_autoplaced yes)
 		(effects
 			(font
@@
 	(label "USB_DP"
 		(at 142.24 71.12 0)
-		(fields_autoplaced yes)
 		(effects
 			(font
@@
 	(label "GPIO15"
 		(at 233.68 101.6 180)
-		(fields_autoplaced yes)
 		(effects
 			(font
@@
 	(label "GPIO10"
 		(at 233.68 88.9 180)
-		(fields_autoplaced yes)
 		(effects
 			(font
@@
 	(label "QSPI_SS"
 		(at 154.94 81.28 0)
-		(fields_autoplaced yes)
 		(effects
 			(font
@@
 	(label "GPIO12"
 		(at 233.68 93.98 180)
-		(fields_autoplaced yes)
 		(effects
 			(font
@@
 	(label "GPIO19"
 		(at 233.68 111.76 180)
-		(fields_autoplaced yes)
 		(effects
 			(font
@@
 	(label "GPIO24"
 		(at 233.68 124.46 180)
-		(fields_autoplaced yes)
 		(effects
 			(font
@@
 	(label "QSPI_SD2"
 		(at 154.94 91.44 0)
-		(fields_autoplaced yes)
 		(effects
 			(font
@@
 	(label "GPIO8"
 		(at 233.68 83.82 180)
-		(fields_autoplaced yes)
 		(effects
 			(font
@@
 	(label "QSPI_SCLK"
 		(at 154.94 96.52 0)
-		(fields_autoplaced yes)
 		(effects
 			(font
@@
 	(label "QSPI_SD3"
 		(at 154.94 93.98 0)
-		(fields_autoplaced yes)
 		(effects
 			(font
@@
 	(label "GPIO17"
 		(at 233.68 106.68 180)
-		(fields_autoplaced yes)
 		(effects
 			(font
@@
 	(label "MCU_1V1"
 		(at 179.07 43.18 0)
-		(fields_autoplaced yes)
 		(effects
 			(font
@@
 	(label "GPIO1"
 		(at 233.68 66.04 180)
-		(fields_autoplaced yes)
 		(effects
 			(font
@@
 	(label "GPIO28_ADC2"
 		(at 233.68 137.16 180)
-		(fields_autoplaced yes)
 		(effects
 			(font
@@
 	(label "GPIO2"
 		(at 233.68 68.58 180)
-		(fields_autoplaced yes)
 		(effects
 			(font
@@
 	(label "GPIO3"
 		(at 233.68 71.12 180)
-		(fields_autoplaced yes)
 		(effects
 			(font
@@
 	(label "GPIO29_ADC3"
 		(at 233.68 139.7 180)
-		(fields_autoplaced yes)
 		(effects
 			(font
@@
 	(label "GPIO25"
 		(at 233.68 127 180)
-		(fields_autoplaced yes)
-		(effects
-			(font
+		(effects
+			(font
