File: hardware/Spartan6_board/pcb.kicad_sch (KiCad schematic)
At the start: 0 parts

Commit message: change DVI FPC pinout to match DVI connector (G-S-S-G), and FPGA device from XC6SLX16-FTG256 to XC6SLX25-3FTG256C
Other:
- title: Glider Lite -> Spartan 6 FPGA board
Changed lines of the file:
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@@
 	(paper "A4")
 	(title_block
-		(title "Glider Lite")
-		(date "2023-12-24")
-		(rev "R0.7")
+		(title "Spartan 6 FPGA board")
+		(date "2026-09-17")
+		(rev "R0.1")
 		(company "Copyright 2023 Modos / Engineer: Wenting Zhang")
 	)

Commit message: review and update manufacturing constraints (via size, etc.)
Other:
- company: Copyright 2023 Modos / Engineer: Wenting Zhang -> (C) 2025-2026 Victor Suarez Rovere <suarezvictor@gmail.com>
Changed lines of the file:
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@@
 	(title_block
 		(title "Spartan 6 FPGA board")
-		(date "2026-09-17")
+		(date "2026-09-18")
 		(rev "R0.1")
-		(company "Copyright 2023 Modos / Engineer: Wenting Zhang")
+		(company "(C) 2025-2026 Victor Suarez Rovere <suarezvictor@gmail.com>")
+		(comment 1 "Copyright 2023 Modos / Engineer: Wenting Zhang")
 	)
 	(text "FPGA DDR Memory"
