File: hardware/Spartan6_board/power.kicad_sch (KiCad schematic)
At the start: 51 parts, among them U1 SY8120, U2 SY8120, U3 SY8120, U4 MT9700, U5 XC6SLX16-FTG256

Commit message: change DVI FPC pinout to match DVI connector (G-S-S-G), and FPGA device from XC6SLX16-FTG256 to XC6SLX25-3FTG256C
Parts:
- U5: value XC6SLX16-FTG256 -> XC6SLX25-3FTG256C; LCSC Part Number C39313 -> C1521716
Other:
- title: Caster EPDC -> Spartan 6 FPGA board
Changed lines of the file:
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@@
 	(paper "A4")
 	(title_block
-		(title "Caster EPDC")
-		(date "2022-07-03")
-		(rev "R0.4")
+		(title "Spartan 6 FPGA board")
+		(date "2026-09-17")
+		(rev "R0.1")
 		(company "Copyright 2022 Modos / Engineer: Wenting Zhang")
 	)
@@
 			)
 		)
-		(property "Value" "XC6SLX16-FTG256"
+		(property "Value" "XC6SLX25-3FTG256C"
 			(at 220.98 48.26 0)
 			(effects
@@
 			)
 		)
-		(property "LCSC Part Number" "C39313"
+		(property "LCSC Part Number" "C1521716"
 			(at 220.98 81.28 0)
 			(effects

Commit message: review and update manufacturing constraints (via size, etc.)
Other:
- company: Copyright 2022 Modos / Engineer: Wenting Zhang -> (C) 2025-2026 Victor Suarez Rovere <suarezvictor@gmail.com>
Changed lines of the file:
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@@
 	(title_block
 		(title "Spartan 6 FPGA board")
-		(date "2026-09-17")
+		(date "2026-09-18")
 		(rev "R0.1")
-		(company "Copyright 2022 Modos / Engineer: Wenting Zhang")
+		(company "(C) 2025-2026 Victor Suarez Rovere <suarezvictor@gmail.com>")
+		(comment 1 "Copyright 2023 Modos / Engineer: Wenting Zhang")
 	)
 	(junction
