File: hardware/Touch_splitter/eDP_touch_adapter_USBHOST.kicad_sch (KiCad schematic)
At the start: 32 parts, among them J1 Conn_01x40, J3 Conn_01x40, J4 USB_B_Micro, U1 RP2354_60QFN, Y1 12MHz

Commit message: add USB host to I2C board based on RP2354 MCU
Parts:
- removed JP3: BOOT, Jumper:SolderJumper-2_P1.3mm_Bridged_RoundedPad1.0x1.5mm, symbol Jumper:SolderJumper_2_Bridged
- added C1: 4.7u 10V, RP2350_60QFN_minimal:C_0402_1005Metric_small_pads, symbol Device:C
- added H1: MountingHole, MountingHole:MountingHole_2.2mm_M2, symbol Mechanical:MountingHole
- added SW1: SW_Push, easyeda2kicad:SW-SMD_4P-L2.5-W1.6-LS2.9_STI-055A12AX, symbol easyeda2kicad:GT-TC194A-H0055-L1
- added TP4, TP5: TestPoint_Small, TestPoint:TestPoint_Pad_D2.0mm, symbol Connector:TestPoint_Small
- J1: value Conn_01x40 -> Conn_01x30; footprint Library:FPC-SMD_40P-P0.50_L4.4-W25.6 -> easyeda2kicad:FPC-SMD_30P-P0.50_FPC-0.5FX-30PWBH15; symbol Connector_Generic_MountingPin:Conn_01x40_MountingPin -> Connector_Generic_MountingPin:Conn_01x30_MountingPin; LCSC Part Number (none) -> C3446034; MPN F0501-B-40-20T-R -> FPC-0.5FX-30PWBH15
- J3: footprint Library:FPC-SMD_40P-P0.50_L4.4-W25.6 -> easyeda2kicad:FPC-SMD_XUNPU_FPC-0.5FX-40PWBH15; LCSC Part Number (none) -> C3446035; MPN F0501-B-40-20T-R -> FPC-0.5FX-40PWBH15
Connections:
- net +3V3: now also C1.1; no longer J1.36 (Pin_36)
- net GND: now also J4.6 (Shield), C1.2, SW1.C; no longer J1.33 (Pin_33)
- net GPIO18: now also J4.4 (ID), TP5.1; no longer J1.40 (Pin_40)
- net GPIO19: now also J1.14 (Pin_14), TP4.1; no longer J1.39 (Pin_39)
- net GPIO20: now also J1.25 (Pin_25); no longer J1.38 (Pin_38)
- net GPIO21: now also J1.24 (Pin_24); no longer J1.37 (Pin_37)
- net MCU_USB_DP: now reaches R8.2, U1.52 (USB_DP)
- net MCU_USB_DN: now reaches R7.2, U1.51 (USB_DM)
- net ~{USB_BOOT} renamed ~{BOOT}
- net ~{BOOT}: now also SW1.A
- no-connect marks 18 -> 11
Other:
- note added: "Special pins in eDP: 1, 24, 25, 30: NC/Reserved 14: Test 17: HPD NOTE USAGE OF pins 24/25 and 14 for I2C"
- moved on the sheet: R7, R8, TP1

Commit message: fixes for producion and notes
Other:
- note added: "TODO: -Add pullups for I2C -Add 3.3V and GND test points -Add "buffer full" signal and an optional LED"
- note added: "This oscillator with 27 ohm works ok"
- note added: "VTSP can work at 3.3V on some panels specified for 5V"
Changed lines of the file:
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@@
+		)
+	)
+	(text "TODO:\n-Add pullups for I2C\n-Add 3.3V and GND test points\n-Add \"buffer full\" signal and an optional LED"
+		(exclude_from_sim no)
+		(at 172.72 40.894 0)
+		(effects
+			(font
+				(size 2 2)
+			)
+			(justify left)
 		)
 	)
@@
 		)
 	)
+	(text "This oscillator\nwith 27 ohm works ok"
+		(exclude_from_sim no)
+		(at 99.314 139.446 0)
+		(effects
+			(font
+				(size 1.27 1.27)
+			)
+			(justify left)
+		)
+	)
 	(text "DECOUPLING"
 		(exclude_from_sim no)
@@
 		)
 	)
+	(text "VTSP can work at 3.3V\non some panels specified for 5V"
+		(exclude_from_sim no)
+		(at 312.674 80.518 0)
+		(effects
+			(font
+				(size 1.27 1.27)
+			)
+			(justify left)
+		)
+	)
